Commit message: new ex12

File: libgex/ex12/urdf/ex12.urdf (robot description, URDF)
Before this commit: robot ex12, 16 links, 15 joints
Links:
- link Link1: mass 0.0217307435979103 -> 0.0229044737579923
- link Link10: mass 0.0265839433569182 -> 0.0193769642321494
- link Link11: mass 0.0230133561838601 -> 0.0215214171982949
- link Link2: mass 0.0220862243589131 -> 0.0242129446909479
- link Link3: mass 0.0195941447971888 -> 0.0220980628650688
- link Link5: mass 0.0178831940703488 -> 0.017883193977129
- link Link6: mass 0.0265839433569186 -> 0.0193769642321485
- link Link7: mass 0.0230133561838601 -> 0.0215214171982948
- link Link9: mass 0.0178831940205361 -> 0.0178831939273071
- link base_link: mass 0.100282584501496 -> 0.104869110532873
Joints:
- joint joint1: origin xyz=0.0726385389055488 -0.00636396103067888 0.0098 rpy=-1.5707963267949 0 -0.785398163397448 -> xyz=0.0751385389055488 -0.00636396103067887 0.0048 rpy=-1.5707963267949 0 -0.785398163397448
- joint joint10: limit lower=-3.14 upper=3.14 effort=10 velocity=3.1 -> lower=-0.7854 upper=1.5708 effort=10 velocity=3.1; origin xyz=0 0 -0.013 rpy=1.5707963267949 -0.192944037979531 0 -> xyz=0 0 -0.013 rpy=1.5707963267949 -0.915757359471054 0
- joint joint11: limit lower=-3.14 upper=3.14 effort=10 velocity=3.1 -> lower=-1.5708 upper=1.5708 effort=10 velocity=3.1; origin xyz=0.0850000000000001 0 0 rpy=0 0 -1.90426963990731 -> xyz=0.0780000000000029 0 0 rpy=0 0 -1.76980911774268
- joint joint12: limit lower=-3.14 upper=3.14 effort=10 velocity=3.1 -> lower=-1.5708 upper=1.5708 effort=10 velocity=3.1; origin xyz=0.0727581521785941 0 0 rpy=3.14159265358979 0 -0.383069500465414 -> xyz=0.0727581521785937 0 0 rpy=3.14159265358979 0 -0.716744568523267
- joint joint13: origin xyz=0 -0.0405 0 rpy=1.5707963267949 0 0 -> xyz=0.0405 0 0 rpy=1.5708 0 0.7854
- joint joint15: origin xyz=0.0405 0 0 rpy=3.1416 0 -1.5708 -> xyz=0.0405000000000056 0 0 rpy=3.14159265358979 0 -1.5707963267949
- joint joint2: limit lower=-3.14 upper=3.14 effort=10 velocity=3.1 -> lower=-1.5708 upper=1.5708 effort=10 velocity=3.1; origin xyz=0 -0.0142 0.0455 rpy=1.5707963267949 -0.785398163397449 -3.14159265358979 -> xyz=0 -0.0192 0.0555 rpy=-1.63723082087563 -1.57079630572147 0.0664344940807344
- joint joint3: limit lower=-3.14 upper=3.14 effort=10 velocity=3.1 -> lower=-1.5708 upper=1.5708 effort=10 velocity=3.1; origin xyz=0.0555 0 0 rpy=0 0 0 -> xyz=0.085 0 0 rpy=0 0 0.713724238084184
- joint joint4: origin xyz=0.0445 0 0 rpy=0 0 0 -> xyz=-0.072758152178594 0 0 rpy=0 0 -2.28452056487908
- joint joint5: limit lower=-3.14 upper=3.14 effort=10 velocity=3.1 -> lower=-1 upper=1 effort=10 velocity=3.1; origin xyz=0.015 0.076293277315303 -0.0509166604983955 rpy=0 0.5235987755983 1.5707963267949 -> xyz=0.0175 0.081459 -0.034 rpy=0 0 1.5708
- joint joint6: limit lower=-3.14 upper=3.14 effort=10 velocity=3.1 -> lower=-0.7854 upper=1.5708 effort=10 velocity=3.1; origin xyz=0 0 0.013 rpy=-1.5707963267949 0.192944037979531 0 -> xyz=0 0 0.013 rpy=-1.5707963267949 0.915757359471054 0
- joint joint7: limit lower=-3.14 upper=3.14 effort=10 velocity=3.1 -> lower=-1.5708 upper=1.5708 effort=10 velocity=3.1; origin xyz=0.0850000000000002 0 0 rpy=0 0 -1.90426963990731 -> xyz=0.0780000000000012 0 0 rpy=0 0 -1.76980911774268
- joint joint8: limit lower=-3.14 upper=3.14 effort=10 velocity=3.1 -> lower=-1.5708 upper=1.5708 effort=10 velocity=3.1; origin xyz=0.0727581521785944 0 0 rpy=3.14159265358979 0 -0.383069500465415 -> xyz=0.0727581521785966 0 0 rpy=3.14159265358979 0 -0.716744568523267
- joint joint9: limit lower=-3.14 upper=3.14 effort=0 velocity=0 -> lower=-1 upper=1 effort=10 velocity=3.1; origin xyz=-0.015 0.076293277315303 -0.0509166604983955 rpy=-3.14159265358979 0.5235987755983 1.5707963267949 -> xyz=-0.0175 0.0814594408408979 -0.034 rpy=3.14159265358979 0 1.5707963267949

Commit message: ex12 direction

File: libgex/ex12/urdf/ex12.urdf (robot description, URDF)
Before this commit: robot EX12, 16 links, 15 joints
Joints:
- joint joint3: limit lower=-1.5708 upper=1.5708 effort=10 velocity=3.1 -> lower=-3.14156 upper=3.14156 effort=10 velocity=3.1
